Commit message: temp commit before clean

File: src/cart_nav_test/urdf/amr_PROPER_acker.urdf.xacro (robot description, xacro)
@@ -505,5 +505,5 @@
         <parent link="base_link" />
         <child link="navsat_link" />
-        <origin xyz="0.1 0 0.135" rpy="0 0 0" />
+        <origin xyz="0.0 0 0.135" rpy="0 0 0" />
     </joint>
     <joint name="base_front_left_steering_joint" type="revolute">
@@ -636,6 +636,6 @@
     <gazebo reference="imu_link">
         <sensor name="imu_sensor" type="imu">
-            <!-- <update_rate>50</update_rate> -->
-            <update_rate>30</update_rate>
+            <update_rate>50</update_rate>
+            <!-- <update_rate>30</update_rate> -->
             <topic>imu</topic>
             <gz_frame_id>imu_link</gz_frame_id>
@@ -677,9 +677,10 @@
             <steering_limit>0.7854</steering_limit>  <!-- radians -->
             <topic>cmd_vel</topic>
-            <odom_topic>odom</odom_topic>
+            <odom_topic>odom_uncorrected</odom_topic>
             <frame_id>odom</frame_id>
-            <!-- <child_frame_id>base_footprint</child_frame_id> -->
-            <child_frame_id>camera_link</child_frame_id>
-            <odom_publish_frequency>30</odom_publish_frequency>
+            <child_frame_id>base_footprint</child_frame_id>
+            <!-- <child_frame_id>camera_link</child_frame_id> -->
+            <!-- <tf_topic>tf</tf_topic> -->
+            <odom_publish_frequency>50</odom_publish_frequency>
         </plugin>
     </gazebo>
